File: SRR-SCHEMATIC/SRR-SCHEMATIC.kicad_pcb (KiCad board)
At the start: 2 copper layers, 206 x 79.1 mm, 54 parts, among them J1 Screw_Terminal_01x02, J2 Conn_01x05, SW2 SW_Push, U1 STM32F411CEUx, U2 NCP1117ST50T3G, U3 NCP1117ST33T3G, U4 NHD-C0220BIZ, U5 VL53L1CXV0FY1, U6 VL53L1CXV0FY1, Y1 16MHz

Commit message: Subindo PCB
Parts:
- added REF**: MountingHole_2.2mm_M2_DIN965, MountingHole:MountingHole_2.2mm_M2_DIN965, F.Cu at (195.3, 111.2)
- added REF**: MountingHole_3.2mm_M3, MountingHole:MountingHole_3.2mm_M3, F.Cu at (103.5, 42.5)
- added REF**: MountingHole_3.2mm_M3, MountingHole:MountingHole_3.2mm_M3, F.Cu at (185.4, 109.2)
- added REF**: MountingHole_2.2mm_M2_DIN965, MountingHole:MountingHole_2.2mm_M2_DIN965, F.Cu at (210.5, 99.1)
- added REF**: MountingHole_3.2mm_M3, MountingHole:MountingHole_3.2mm_M3, F.Cu at (103.5, 109.2)
- added REF**: MountingHole_3.2mm_M3, MountingHole:MountingHole_3.2mm_M3, F.Cu at (185.4, 41.9)
- added REF**: MountingHole_2.2mm_M2_DIN965, MountingHole:MountingHole_2.2mm_M2_DIN965, F.Cu at (210.8, 79.4)
- added REF**: MountingHole_2.2mm_M2_DIN965, MountingHole:MountingHole_2.2mm_M2_DIN965, F.Cu at (195.6, 91.4)
- moved C6 69.6 mm to (194.9, 101.4)
- moved R4 69.6 mm to (201.3, 106.0)
- moved C4 69.6 mm to (197.4, 101.4)
- moved R2 69.6 mm to (205.8, 101.5)
- moved R3 69.6 mm to (196.1, 106.1)
- moved R9 69.6 mm to (206.2, 106.1)
- moved U6 69.6 mm to (201.6, 101.6)
- moved ConnLaserMC2 67.6 mm to (203.1, 110.5)
- moved C13 50.2 mm to (198.1, 81.1), turned to 90 degrees
- moved ConnLaser1MC1 48.7 mm to (203.6, 90.8), turned to 90 degrees
- moved R10 47.3 mm to (196.2, 86.4), turned to 0 degrees
- moved C11 46.2 mm to (195.6, 81.1), turned to 90 degrees
- moved U5 45.8 mm to (202.6, 81.3)
- moved R12 45.5 mm to (201.9, 86.4), turned to 180 degrees
- moved R8 44.1 mm to (207.0, 81.3), turned to 90 degrees
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- renumbered ConnMCLaser3 to ConnLaserMC2
Other:
- board size 206 x 79.1 mm -> 113.9 x 75.4 mm

Commit message: Subindo codigo e PCB
Parts:
- J1: moved to F.Cu
- moved F1 14.1 mm to (113.2, 94.9)
- moved C21 13.3 mm to (139.1, 75.0)
- moved R17 6.57 mm to (138.0, 81.0)
- moved J1 6.41 mm to (105.1, 84.7), turned to -90 degrees
- moved C23 4.42 mm to (133.8, 80.8), turned to 90 degrees
- moved Y1 2.54 mm to (132.9, 75.4), turned to 180 degrees
- moved R4 0.91 mm to (200.5, 106.5), turned to 0 degrees
- moved R12 0.79 mm to (201.5, 87.0), turned to 0 degrees
- renumbered ConnLaserMC2 to ConnLaser2MC1
Connections:
- ConnLaser2MC1 pad 2: Net-(ConnMCLaser3-Pad2) -> Net-(ConnLaser2MC1-Pad2)
- ConnLaser2MC1 pad 3: Net-(ConnMCLaser3-Pad3) -> Net-(ConnLaser2MC1-Pad3)
- ConnMCLaser1 pad 2: I2C1_SCL_LASER1 -> I2C1_SDA_LASER1
- ConnMCLaser1 pad 3: I2C1_SDA_LASER1 -> I2C1_SCL_LASER1
- ConnMCLaser2 pad 2: I2C2_SCL_LASER2 -> I2C2_SDA_LASER2
- ConnMCLaser2 pad 3: I2C2_SDA_LASER2 -> I2C2_SCL_LASER2
- R10 pad 2: Net-(ConnLaser1MC1-Pad2) -> Net-(ConnLaser1MC1-Pad3)
- R12 pad 2: Net-(ConnLaser1MC1-Pad3) -> Net-(ConnLaser1MC1-Pad2)
- R3 pad 2: Net-(ConnMCLaser3-Pad2) -> Net-(ConnLaser2MC1-Pad3)
- R4 pad 2: Net-(ConnMCLaser3-Pad3) -> Net-(ConnLaser2MC1-Pad2)
- U5 pad 10: Net-(ConnLaser1MC1-Pad2) -> Net-(ConnLaser1MC1-Pad3)
- U5 pad 9: Net-(ConnLaser1MC1-Pad3) -> Net-(ConnLaser1MC1-Pad2)
- U6 pad 10: Net-(ConnMCLaser3-Pad2) -> Net-(ConnLaser2MC1-Pad3)
- U6 pad 9: Net-(ConnMCLaser3-Pad3) -> Net-(ConnLaser2MC1-Pad2)

Commit message: Subindo PCB Corrigida
Parts:
- Laser1: renamed from ConnMCLaser1; footprint Connector_PinHeader_1.00mm:PinHeader_1x05_P1.00mm_Vertical -> Connector_PinHeader_2.54mm:PinHeader_1x05_P2.54mm_Vertical
- Laser1: renamed from ConnLaser1MC1; footprint Connector_PinHeader_1.00mm:PinHeader_1x05_P1.00mm_Vertical -> Connector_PinHeader_2.54mm:PinHeader_1x05_P2.54mm_Vertical
- Laser2: renamed from ConnLaser2MC1; footprint Connector_PinHeader_1.00mm:PinHeader_1x05_P1.00mm_Vertical -> Connector_PinHeader_2.54mm:PinHeader_1x05_P2.54mm_Vertical
- Laser2: renamed from ConnMCLaser2; footprint Connector_PinHeader_1.00mm:PinHeader_1x05_P1.00mm_Vertical -> Connector_PinHeader_2.54mm:PinHeader_1x05_P2.54mm_Vertical
- STLINK: renamed from J2; footprint Connector_PinHeader_1.00mm:PinHeader_1x05_P1.00mm_Vertical -> Connector_PinHeader_2.54mm:PinHeader_1x05_P2.54mm_Vertical
- moved R7 30.2 mm to (145.4, 77.8), turned to 90 degrees
- moved R6 22.9 mm to (149.4, 74.3), turned to 0 degrees
- moved R17 19.0 mm to (155.6, 88.3), turned to 90 degrees
- moved F1 18.9 mm to (120.7, 77.5)
- moved Y1 18.6 mm to (149.2, 84.5), turned to -90 degrees
- moved C23 17.1 mm to (149.2, 88.3), turned to 180 degrees
- moved D6 16.7 mm to (138.0, 92.1)
- moved R12 15.3 mm to (202.3, 71.8)
- moved R4 15.1 mm to (201.7, 91.4)
- moved REF** 14.9 mm to (106.7, 94.6)
- moved Laser1 14.7 mm to (200.6, 76.4)
- moved Laser2 14.7 mm to (200.4, 96.1)
- moved C11 14.6 mm to (195.9, 66.5)
- moved C13 14.6 mm to (198.5, 66.5)
- moved C4 14.6 mm to (197.8, 86.8)
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Connections:
- Laser1 pad 2: I2C1_SDA_LASER1 -> I2C1_SCL_LASER1
- Laser1 pad 3: I2C1_SCL_LASER1 -> I2C1_SDA_LASER1
- R10 pad 2: Net-(ConnLaser1MC1-Pad3) -> Net-(ConnLaser1MC1-Pad2)
- R12 pad 2: Net-(ConnLaser1MC1-Pad2) -> Net-(ConnLaser1MC1-Pad3)
- U1 pad 13: RESET_NHD -> unconnected-(U1-Pad13)
- U1 pad 29: unconnected-(U1-Pad29) -> I2C3_SCL_NHD
- U1 pad 45: I2C3_SCL_NHD -> RESET_NHD
- U5 pad 10: Net-(ConnLaser1MC1-Pad3) -> Net-(ConnLaser1MC1-Pad2)
- U5 pad 9: Net-(ConnLaser1MC1-Pad2) -> Net-(ConnLaser1MC1-Pad3)
Routing:
- net +3V3: track 0.00 -> 189.5 mm, vias 0 -> 7
- net +3.3VADC: track 0.00 -> 50.5 mm
- net +3.3VDAC: track 0.00 -> 49.3 mm
- net Net-(C1-Pad1): track 0.00 -> 39.6 mm
- net GPIO1_LASER1: track 0.00 -> 37.3 mm, vias 0 -> 1
- net I2C3_SDA_NHD: track 0.00 -> 32.6 mm, vias 0 -> 2
- net I2C3_SCL_NHD: track 0.00 -> 32.0 mm, vias 0 -> 2
- net I2C1_SDA_LASER1: track 0.00 -> 26.4 mm
- net GNDREF: track 0.00 -> 25.8 mm, vias 0 -> 44
- net +5V: track 0.00 -> 25.4 mm, vias 0 -> 2
- net I2C1_SCL_LASER1: track 0.00 -> 24.7 mm
- net I2C2_SDA_LASER2: track 0.00 -> 23.5 mm
- net GPIO1_LASER2: track 0.00 -> 23.5 mm
- net I2C2_SCL_LASER2: track 0.00 -> 22.6 mm
- net DISTANCE_REGULATOR: track 0.00 -> 18.9 mm
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- added copper zone on B.Cu, net GND
- added copper zone on F.Cu, net GND
- added copper zone on B.Cu, net GND2
- added copper zone on F.Cu, net GND2
- added copper zone on B.Cu, net GNDREF
- added copper zone on F.Cu, net GNDREF
Other:
- board size 113.9 x 75.4 mm -> 112 x 65.9 mm
- board text added: "GND"
- board text added: "GPIO"
- board text added: "SCL"
- board text added: "SDA"
- board text added: "SWCLK"
- board text added: "SWDIO"
- board text added: "VCC"
