File: SRR-SCHEMATIC/SRR-SCHEMATIC.kicad_sch (KiCad schematic)
At the start: 54 parts, among them J1 Screw_Terminal_01x02, J2 Conn_01x05, SW2 SW_Push, U1 STM32F411CEUx, U2 NCP1117ST50T3G, U3 NCP1117ST33T3G, U4 NHD-C0220BIZ, U5 VL53L1CXV0FY1, U6 VL53L1CXV0FY1, Y1 16MHz

Commit message: Subindo PCB
Parts:
- renumbered ConnMCLaser3 to ConnLaser2MC
Changed lines of the file:
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@@
   (symbol (lib_id "Connector_Generic:Conn_01x05") (at 297.18 43.18 180) (unit 1)
     (in_bom yes) (on_board yes)
-    (property "Reference" "ConnMCLaser3" (id 0) (at 297.18 31.75 0))
+    (property "Reference" "ConnLaser2MC" (id 0) (at 297.18 31.75 0))
     (property "Value" "Conn_01x05" (id 1) (at 297.18 34.29 0))
     (property "Footprint" "Connector_PinHeader_1.00mm:PinHeader_1x05_P1.00mm_Vertical" (id 2) (at 297.18 43.18 0)
@@
       (reference "ConnLaser1MC1") (unit 1) (value "Conn_01x05") (footprint "Connector_PinHeader_1.00mm:PinHeader_1x05_P1.00mm_Vertical")
     )
+    (path "/c9380cc6-4b6e-48d8-9be0-bc8c792749c5"
+      (reference "ConnLaser2MC") (unit 1) (value "Conn_01x05") (footprint "Connector_PinHeader_1.00mm:PinHeader_1x05_P1.00mm_Vertical")
+    )
     (path "/4253a868-8f08-4479-a46f-7ca68e6be92e"
       (reference "ConnMCLaser1") (unit 1) (value "Conn_01x05") (footprint "Connector_PinHeader_1.00mm:PinHeader_1x05_P1.00mm_Vertical")
@@
       (reference "ConnMCLaser2") (unit 1) (value "Conn_01x05") (footprint "Connector_PinHeader_1.00mm:PinHeader_1x05_P1.00mm_Vertical")
     )
-    (path "/c9380cc6-4b6e-48d8-9be0-bc8c792749c5"
-      (reference "ConnMCLaser3") (unit 1) (value "Conn_01x05") (footprint "Connector_PinHeader_1.00mm:PinHeader_1x05_P1.00mm_Vertical")
-    )
     (path "/04180427-de75-4b3b-9aee-00b35268037e"

Commit message: Subindo codigo e PCB
Parts:
- renumbered ConnLaser2MC to ConnLaser2MC1
Connections:
- net I2C1_SCL_LASER1: now also ConnMCLaser1.3 (Pin_3); no longer ConnMCLaser1.2 (Pin_2)
- net I2C1_SDA_LASER1: now also ConnMCLaser1.2 (Pin_2); no longer ConnMCLaser1.3 (Pin_3)
- net I2C2_SCL_LASER2: now also ConnMCLaser2.3 (Pin_3); no longer ConnMCLaser2.2 (Pin_2)
- net I2C2_SDA_LASER2: now also ConnMCLaser2.2 (Pin_2); no longer ConnMCLaser2.3 (Pin_3)
- net at R10.2, U5.10 (SCL): now also ConnLaser1MC1.3 (Pin_3); no longer ConnLaser1MC1.2 (Pin_2)
- net at R12.2, U5.9 (SDA): now also ConnLaser1MC1.2 (Pin_2); no longer ConnLaser1MC1.3 (Pin_3)
- net at R3.2, U6.10 (SCL): now also ConnLaser2MC1.3 (Pin_3); no longer ConnLaser2MC1.2 (Pin_2)
- net at R4.2, U6.9 (SDA): now also ConnLaser2MC1.2 (Pin_2); no longer ConnLaser2MC1.3 (Pin_3)
Changed lines of the file:
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@@
   (junction (at 341.63 194.31) (diameter 0) (color 0 0 0 0)
   )
-  (junction (at 334.01 43.18) (diameter 0) (color 0 0 0 0)
-  )
   (junction (at 283.21 220.98) (diameter 0) (color 0 0 0 0)
   )
@@
   (junction (at 379.73 59.69) (diameter 0) (color 0 0 0 0)
   )
+  (junction (at 334.01 43.18) (diameter 0) (color 0 0 0 0)
+  )
   (junction (at 72.39 215.9) (diameter 0) (color 0 0 0 0)
   )
@@
   (junction (at 270.51 220.98) (diameter 0) (color 0 0 0 0)
   )
-  (junction (at 330.2 45.72) (diameter 0) (color 0 0 0 0)
-  )
   (junction (at 43.18 96.52) (diameter 0) (color 0 0 0 0)
   )
@@
   (junction (at 48.26 109.22) (diameter 0) (color 0 0 0 0)
   )
+  (junction (at 330.2 45.72) (diameter 0) (color 0 0 0 0)
+  )
   (junction (at 270.51 234.95) (diameter 0) (color 0 0 0 0)
   )
@@
     (stroke (width 0) (type default) (color 0 0 0 0))
   )
+  (wire (pts (xy 317.5 43.18) (xy 317.5 45.72))
+    (stroke (width 0) (type default) (color 0 0 0 0))
+  )
   (wire (pts (xy 143.51 96.52) (xy 127 96.52))
     (stroke (width 0) (type default) (color 0 0 0 0))
@@
     (stroke (width 0) (type default) (color 0 0 0 0))
   )
+  (wire (pts (xy 320.04 45.72) (xy 320.04 44.45))
+    (stroke (width 0) (type default) (color 0 0 0 0))
+  )
+  (wire (pts (xy 312.42 44.45) (xy 312.42 43.18))
+    (stroke (width 0) (type default) (color 0 0 0 0))
+  )
   (wire (pts (xy 379.73 38.1) (xy 379.73 35.56))
     (stroke (width 0) (type default) (color 0 0 0 0))
@@
     (stroke (width 0) (type default) (color 0 0 0 0))
   )
+  (wire (pts (xy 302.26 43.18) (xy 312.42 43.18))
+    (stroke (width 0) (type default) (color 0 0 0 0))
+  )
   (wire (pts (xy 374.65 19.05) (xy 374.65 26.67))
     (stroke (width 0) (type default) (color 0 0 0 0))
@@
     (stroke (width 0) (type default) (color 0 0 0 0))
   )
-  (wire (pts (xy 302.26 45.72) (xy 330.2 45.72))
-    (stroke (width 0) (type default) (color 0 0 0 0))
-  )
   (wire (pts (xy 219.71 19.05) (xy 219.71 21.59))
     (stroke (width 0) (type default) (color 0 0 0 0))
@@
     (stroke (width 0) (type default) (color 0 0 0 0))
   )
+  (wire (pts (xy 334.01 43.18) (xy 317.5 43.18))
+    (stroke (width 0) (type default) (color 0 0 0 0))
+  )
   (wire (pts (xy 241.3 29.21) (xy 266.7 29.21))
     (stroke (width 0) (type default) (color 0 0 0 0))
@@
     (stroke (width 0) (type default) (color 0 0 0 0))
   )
+  (wire (pts (xy 302.26 45.72) (xy 317.5 45.72))
+    (stroke (width 0) (type default) (color 0 0 0 0))
+  )
   (wire (pts (xy 243.84 220.98) (xy 257.81 220.98))
     (stroke (width 0) (type default) (color 0 0 0 0))
@@
     (stroke (width 0) (type default) (color 0 0 0 0))
   )
+  (wire (pts (xy 320.04 45.72) (xy 330.2 45.72))
+    (stroke (width 0) (type default) (color 0 0 0 0))
+  )
   (wire (pts (xy 217.17 45.72) (xy 228.6 45.72))
     (stroke (width 0) (type default) (color 0 0 0 0))
@@
     (stroke (width 0) (type default) (color 0 0 0 0))
   )
-  (wire (pts (xy 205.74 41.91) (xy 208.28 41.91))
-    (stroke (width 0) (type default) (color 0 0 0 0))
-  )
   (wire (pts (xy 217.17 21.59) (xy 219.71 21.59))
     (stroke (width 0) (type default) (color 0 0 0 0))
@@
     (stroke (width 0) (type default) (color 0 0 0 0))
   )
+  (wire (pts (xy 185.42 40.64) (xy 196.85 40.64))
+    (stroke (width 0) (type default) (color 0 0 0 0))
+  )
   (wire (pts (xy 278.13 35.56) (xy 278.13 38.1))
     (stroke (width 0) (type default) (color 0 0 0 0))
   )
+  (wire (pts (xy 320.04 44.45) (xy 312.42 44.45))
+    (stroke (width 0) (type default) (color 0 0 0 0))
+  )
   (wire (pts (xy 106.68 208.28) (xy 106.68 210.82))
     (stroke (width 0) (type default) (color 0 0 0 0))
@@
     (stroke (width 0) (type default) (color 0 0 0 0))
   )
-  (wire (pts (xy 302.26 43.18) (xy 334.01 43.18))
+  (wire (pts (xy 191.77 43.18) (xy 185.42 43.18))
     (stroke (width 0) (type default) (color 0 0 0 0))
   )
@@
     (stroke (width 0) (type default) (color 0 0 0 0))
   )
-  (wire (pts (xy 205.74 41.91) (xy 205.74 40.64))
+  (wire (pts (xy 200.66 208.28) (xy 200.66 209.55))
     (stroke (width 0) (type default) (color 0 0 0 0))
   )
-  (wire (pts (xy 200.66 208.28) (xy 200.66 209.55))
+  (wire (pts (xy 191.77 41.91) (xy 191.77 43.18))
     (stroke (width 0) (type default) (color 0 0 0 0))
   )
@@
     (stroke (width 0) (type default) (color 0 0 0 0))
   )
-  (wire (pts (xy 326.39 36.83) (xy 326.39 49.53))
-    (stroke (width 0) (type default) (color 0 0 0 0))
-  )
   (wire (pts (xy 114.3 35.56) (xy 127 35.56))
     (stroke (width 0) (type default) (color 0 0 0 0))
@@
     (stroke (width 0) (type default) (color 0 0 0 0))
   )
-  (wire (pts (xy 205.74 40.64) (xy 185.42 40.64))
-    (stroke (width 0) (type default) (color 0 0 0 0))
-  )
   (wire (pts (xy 337.82 132.08) (xy 337.82 138.43))
     (stroke (width 0) (type default) (color 0 0 0 0))
@@
     (stroke (width 0) (type default) (color 0 0 0 0))
   )
+  (wire (pts (xy 205.74 43.18) (xy 196.85 43.18))
+    (stroke (width 0) (type default) (color 0 0 0 0))
+  )
   (wire (pts (xy 344.17 128.27) (xy 344.17 132.08))
     (stroke (width 0) (type default) (color 0 0 0 0))
@@
     (stroke (width 0) (type default) (color 0 0 0 0))
   )
-  (wire (pts (xy 205.74 43.18) (xy 185.42 43.18))
+  (wire (pts (xy 391.16 35.56) (xy 391.16 38.1))
     (stroke (width 0) (type default) (color 0 0 0 0))
   )
-  (wire (pts (xy 391.16 35.56) (xy 391.16 38.1))
+  (wire (pts (xy 196.85 43.18) (xy 196.85 40.64))
     (stroke (width 0) (type default) (color 0 0 0 0))
   )
@@
     (stroke (width 0) (type default) (color 0 0 0 0))
   )
+  (wire (pts (xy 191.77 41.91) (xy 208.28 41.91))
+    (stroke (width 0) (type default) (color 0 0 0 0))
+  )
+  (wire (pts (xy 326.39 36.83) (xy 326.39 49.53))
+    (stroke (width 0) (type default) (color 0 0 0 0))
+  )
   (wire (pts (xy 270.51 231.14) (xy 270.51 234.95))
     (stroke (width 0) (type default) (color 0 0 0 0))
@@
     )
   )
-  (global_label "I2C2_SCL_LASER2" (shape input) (at 210.82 242.57 0) (fields_autoplaced)
+  (global_label "I2C2_SCL_LASER2" (shape input) (at 209.55 237.49 0) (fields_autoplaced)
     (effects (font (size 1.27 1.27)) (justify left))
-    (property "Intersheet References" "${INTERSHEET_REFS}" (id 0) (at 229.9245 242.6494 0)
+    (property "Intersheet References" "${INTERSHEET_REFS}" (id 0) (at 228.6545 237.5694 0)
       (effects (font (size 1.27 1.27)) (justify left) hide)
     )
@@
     )
   )
-  (global_label "I2C2_SDA_LASER2" (shape input) (at 209.55 237.49 0) (fields_autoplaced)
+  (global_label "I2C2_SDA_LASER2" (shape input) (at 210.82 242.57 0) (fields_autoplaced)
     (effects (font (size 1.27 1.27)) (justify left))
-    (property "Intersheet References" "${INTERSHEET_REFS}" (id 0) (at 228.715 237.5694 0)
+    (property "Intersheet References" "${INTERSHEET_REFS}" (id 0) (at 229.985 242.6494 0)
       (effects (font (size 1.27 1.27)) (justify left) hide)
     )
@@
     )
   )
-  (global_label "I2C1_SCL_LASER1" (shape input) (at 208.28 215.9 0) (fields_autoplaced)
+  (global_label "I2C1_SCL_LASER1" (shape input) (at 208.28 212.09 0) (fields_autoplaced)
     (effects (font (size 1.27 1.27)) (justify left))
-    (property "Intersheet References" "${INTERSHEET_REFS}" (id 0) (at 227.3845 215.9794 0)
+    (property "Intersheet References" "${INTERSHEET_REFS}" (id 0) (at 227.3845 212.1694 0)
       (effects (font (size 1.27 1.27)) (justify left) hide)
     )
@@
     )
   )
-  (global_label "I2C1_SDA_LASER1" (shape input) (at 208.28 212.09 0) (fields_autoplaced)
+  (global_label "I2C1_SDA_LASER1" (shape input) (at 208.28 215.9 0) (fields_autoplaced)
     (effects (font (size 1.27 1.27)) (justify left))
-    (property "Intersheet References" "${INTERSHEET_REFS}" (id 0) (at 227.445 212.0106 0)
+    (property "Intersheet References" "${INTERSHEET_REFS}" (id 0) (at 227.445 215.8206 0)
       (effects (font (size 1.27 1.27)) (justify left) hide)
     )
@@
   (symbol (lib_id "Connector_Generic:Conn_01x05") (at 297.18 43.18 180) (unit 1)
     (in_bom yes) (on_board yes)
-    (property "Reference" "ConnLaser2MC" (id 0) (at 297.18 31.75 0))
+    (property "Reference" "ConnLaser2MC1" (id 0) (at 297.18 31.75 0))
     (property "Value" "Conn_01x05" (id 1) (at 297.18 34.29 0))
     (property "Footprint" "Connector_PinHeader_1.00mm:PinHeader_1x05_P1.00mm_Vertical" (id 2) (at 297.18 43.18 0)
@@
     )
     (path "/c9380cc6-4b6e-48d8-9be0-bc8c792749c5"
-      (reference "ConnLaser2MC") (unit 1) (value "Conn_01x05") (footprint "Connector_PinHeader_1.00mm:PinHeader_1x05_P1.00mm_Vertical")
+      (reference "ConnLaser2MC1") (unit 1) (value "Conn_01x05") (footprint "Connector_PinHeader_1.00mm:PinHeader_1x05_P1.00mm_Vertical")
     )
     (path "/4253a868-8f08-4479-a46f-7ca68e6be92e"

Commit message: Subindo PCB Corrigida
Parts:
- ConnLaser1MC1, ConnLaser2MC1, ConnMCLaser1, ConnMCLaser2, J2: footprint Connector_PinHeader_1.00mm:PinHeader_1x05_P1.00mm_Vertical -> Connector_PinHeader_2.54mm:PinHeader_1x05_P2.54mm_Vertical
Connections:
- net I2C1_SCL_LASER1: now also ConnMCLaser1.2 (Pin_2); no longer ConnMCLaser1.3 (Pin_3)
- net I2C1_SDA_LASER1: now also ConnMCLaser1.3 (Pin_3); no longer ConnMCLaser1.2 (Pin_2)
- net I2C3_SCL_NHD: now also U1.29 (PA8); no longer U1.45 (PB8)
- net RESET_NHD: now also U1.45 (PB8); no longer U1.13 (PA3)
- net at R10.2, U5.10 (SCL): now also ConnLaser1MC1.2 (Pin_2); no longer ConnLaser1MC1.3 (Pin_3)
- net at R12.2, U5.9 (SDA): now also ConnLaser1MC1.3 (Pin_3); no longer ConnLaser1MC1.2 (Pin_2)
